File: hardware/odri-power-board.kicad_sch (KiCad schematic)
At the start: 55 parts, among them IC1 LTC7001IMSE#PBF, J1 PROG, J10 OUT, J11 OUT, J12 OUT, J13 SW, J2 SPI, J3 IN, J4 OUT, J5 OUT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

Commit message: add mounting holes and silkscreen
Parts:
- D1, D2: DigiKey (none) -> 1568-COM-16347CT-ND; Part No (none) -> COM-16347
Changed lines of the file:
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@@
+			)
+		)
+		(property "DigiKey" "1568-COM-16347CT-ND"
+			(at 147.32 35.56 0)
+			(effects
+				(font
+					(size 1.27 1.27)
+				)
+				(hide yes)
+			)
+		)
+		(property "Part No" "COM-16347"
+			(at 147.32 35.56 0)
+			(effects
+				(font
+					(size 1.27 1.27)
+				)
+				(hide yes)
 			)
 		)
@@
 			(at 162.56 35.56 0)
 			(effects
+				(font
+					(size 1.27 1.27)
+				)
+				(hide yes)
+			)
+		)
+		(property "DigiKey" "1568-COM-16347CT-ND"
+			(at 162.56 35.56 0)
+			(effects
+				(font
+					(size 1.27 1.27)
+				)
+				(hide yes)
+			)
+		)
+		(property "Part No" "COM-16347"
+			(at 162.56 35.56 0)
+			(effects
